File: hardware/carambola2-inair9-io-shield/ioshield.brd (EAGLE design)
At the start: 65.1 x 65 mm, 79 parts, among them IC1 PCF8591P, IC2 LM336LP, J1 I2C: RTC module, J10 RST, J12 Carambola2 J12, J13 Carambola2 J13, J2 22-23-2101, J3 inAir9-GND-wing, J4 inAir9 wing 2, J5 BMP180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

Commit message: Schematics as provided to OshPark
Parts:
- added R17, R18: 10K, rcl:M1206
Connections:
- net GND: now also R17.1, R18.1
- net MISO: now also R17.2
- net MOSI: now also R18.2
Routing:
- net GND: track 238.8 -> 242.8 mm, vias 0 -> 1
- net MOSI: track 21.7 -> 22.5 mm
- net MISO: track 26.9 -> 27.7 mm
Changed lines of the file:
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@@
 <attribute name="VALUE" x="59.182" y="39.97" size="0.0254" layer="27"/>
+</element>
+<element name="R17" library="rcl" package="M1206" value="10K" x="67.945" y="25.4" smashed="yes" rot="MR270">
+<attribute name="NAME" x="66.675" y="26.035" size="1.016" layer="26" rot="MR270"/>
+</element>
+<element name="R18" library="rcl" package="M1206" value="10K" x="55.245" y="27.94" smashed="yes" rot="MR225">
+<attribute name="NAME" x="57.939075" y="28.838025" size="1.016" layer="26" rot="MR225"/>
 </element>
 </elements>
@@
 </polygon>
 <wire x1="20.0724" y1="35.6792" x2="20.066" y2="35.052" width="0.6096" layer="1"/>
+<contactref element="R17" pad="1"/>
+<contactref element="R18" pad="1"/>
+<via x="51.435" y="31.75" extent="1-16" drill="0.6096" diameter="1.016"/>
+<wire x1="54.255053125" y1="28.929946875" x2="51.435" y2="31.75" width="0.4064" layer="16"/>
 </signal>
 <signal name="+3V3">
@@
 <wire x1="65.405" y1="30.1625" x2="67.31" y2="32.0675" width="0.254" layer="16"/>
 <wire x1="60.6425" y1="30.1625" x2="65.405" y2="30.1625" width="0.254" layer="16"/>
-<wire x1="55.245" y1="24.765" x2="60.6425" y2="30.1625" width="0.254" layer="16"/>
+<wire x1="55.245" y1="24.765" x2="56.8325" y2="26.3525" width="0.254" layer="16"/>
+<wire x1="56.8325" y1="26.3525" x2="60.6425" y2="30.1625" width="0.254" layer="16"/>
 <wire x1="52.3875" y1="21.9075" x2="55.245" y2="24.765" width="0.254" layer="1"/>
 <wire x1="52.3875" y1="20.32" x2="52.3875" y2="21.9075" width="0.254" layer="16"/>
@@
 <via x="55.245" y="24.765" extent="1-16" drill="0.6096"/>
 <via x="52.3875" y="21.9075" extent="1-16" drill="0.6096"/>
+<contactref element="R18" pad="2"/>
+<wire x1="56.23495" y1="26.95005" x2="56.8325" y2="26.3525" width="0.4064" layer="16"/>
 </signal>
 <signal name="MISO">
@@
 <contactref element="J4" pad="4"/>
 <wire x1="69.85" y1="24.765" x2="69.85" y2="32.258" width="0.254" layer="1"/>
-<wire x1="65.7225" y1="20.6375" x2="69.85" y2="24.765" width="0.254" layer="16"/>
+<wire x1="65.7225" y1="20.6375" x2="68.58" y2="23.495" width="0.254" layer="16"/>
+<wire x1="68.58" y1="23.495" x2="69.85" y2="24.765" width="0.254" layer="16"/>
 <wire x1="65.7225" y1="19.3675" x2="65.7225" y2="20.6375" width="0.254" layer="16"/>
 <wire x1="64.77" y1="18.415" x2="65.7225" y2="19.3675" width="0.254" layer="16"/>
@@
 <wire x1="54.61" y1="19.685" x2="54.356" y2="19.822" width="0.254" layer="16"/>
 <via x="69.85" y="24.765" extent="1-16" drill="0.6096"/>
+<contactref element="R17" pad="2"/>
+<wire x1="67.945" y1="24" x2="68.58" y2="23.495" width="0.4064" layer="16"/>
 </signal>
 <signal name="AGND">
